Commit message: slam working

File: container/launch-content/parameters/bento-box-neo.urdf (robot description, URDF)
Before this commit: robot bento-box-neo, 10 links, 9 joints
Joints:
- joint base_joint: child base_footprint -> base_link; origin xyz=0.0 0.0 ${-(wheel_radius+wheel_zoff)} rpy=0 0 0 -> xyz=0.0 0.0 ${wheel_radius+wheel_zoff} rpy=0 0 0; parent base_link -> base_footprint

Commit message: update arm urdf - gripper

File: container/launch-content/parameters/bento-box-neo.urdf (robot description, URDF)
Before this commit: robot bento-box-neo, 10 links, 9 joints
Links:
- added link arm_endeffector_link; visual box size=${gripper_part_length} ${parts_width/2} ${parts_height/2}
- added link arm_endeffector_link_2; visual box size=${gripper_part_length} ${parts_width/2} ${parts_height/2}
- link arm_wrist_link: geometry visual box size=${wrist_part_length} ${parts_width} ${parts_height}
Joints:
- added joint arm_endeffector_joint: type revolute, parent arm_wrist_link, child arm_endeffector_link, origin xyz=${wrist_part_length} ${parts_width/4} ${parts_height/2} rpy=0 0 0, axis 0 0 1, limit lower=0.0 upper=3.7692 effort=1000.0 velocity=0.5
- added joint arm_endeffector_joint_2: type revolute, parent arm_wrist_link, child arm_endeffector_link_2, origin xyz=${wrist_part_length} ${-parts_width/4} ${parts_height/2} rpy=0 0 0, axis 0 0 1, limit lower=0.0 upper=3.7692 effort=1000.0 velocity=0.5, mimic joint=arm_endeffector_joint multiplier=-1.0 offset=0.0
